Commit message: meshes path

File: coppelia/urdf/mazebot/mazebot.urdf (robot description, URDF)
Before this commit: robot PioneerP3DX__158__, 5 links, 4 joints
Links:
- link PioneerP3DX__158__: geometry collision mesh filename=package://mazebot/models/mazebot_PioneerP3DX__158__.dae; visual mesh filename=package://mazebot/models/mazebot_visible__171__.dae
- link caster_link__166__: geometry collision cylinder length=0.0014799622585997 radius=0.0088369632139802; visual mesh filename=package://mazebot/models/mazebot_caster_link_visible__170__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
- link leftWheel__163__: geometry collision cylinder length=0.025000000372529 radius=0.048749998211861; visual mesh filename=package://mazebot/models/mazebot_leftWheel_visible__164__.d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
- link rightWheel__160__: geometry collision cylinder length=0.025000000372529 radius=0.048749998211861; visual mesh filename=package://mazebot/models/mazebot_rightWheel_visible__161__.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

Commit message: Rename base_link to base_link in .urdf files

File: coppelia/urdf/mazebot/mazebot.urdf (robot description, URDF)
Before this commit: robot PioneerP3DX__158__, 5 links, 4 joints
Links:
- removed link PioneerP3DX__158__
- added link base_link, mass 2.0; collision mesh filename=package://mazebot/models/mazebot_PioneerP3DX__158__.dae; visual mesh filename=package://mazebot/models/mazebot_visible__171__.dae
Joints:
- joint caster_freeJoint__165__: parent PioneerP3DX__158__ -> base_link
- joint leftMotor__162__: parent PioneerP3DX__158__ -> base_link
- joint rightMotor__159__: parent PioneerP3DX__158__ -> base_link
