Commit message: Mazebot urdf with laser

File: coppelia/urdf/mazebotV0/mazebot.urdf (robot description, URDF)
Before this commit: robot PioneerP3DX__135__, 5 links, 4 joints
Links:
- removed link caster_link__143__
- removed link caster_wheel__145__
- removed link leftWheel__140__
- removed link rightWheel__137__
- added link caster_link__166__, mass 0.125; collision cylinder length=0.0014799622585997 radius=0.0088369632139802; visual mesh filename=package://mazebot/models/mazebot_caster_link_visible__170__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
- added link caster_wheel__168__, mass 0.03125; collision cylinder length=0.0025899142492563 radius=0.014799509197474; visual cylinder length=0.010359656997025 radius=0.014799509197474
- added link leftWheel__163__, mass 0.1875; collision cylinder length=0.025000000372529 radius=0.048749998211861; visual mesh filename=package://mazebot/models/mazebot_leftWheel_visible__164__.d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
- added link rightWheel__160__, mass 0.1875; collision cylinder length=0.025000000372529 radius=0.048749998211861; visual mesh filename=package://mazebot/models/mazebot_rightWheel_visible__161__.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
- link base_link: geometry collision mesh filename=package://mazebot/models/mazebot_PioneerP3DX__158__.dae; visual mesh filename=package://mazebot/models/mazebot_visible__171__.dae
Joints:
- removed joint caster_freeJoint__142__
- removed joint caster_freeJoint__144__
- removed joint leftMotor__139__
- removed joint rightMotor__136__
- added joint caster_freeJoint__165__: type continuous, parent base_link, child caster_link__166__, origin xyz=-0.074513 -0.000001 -0.038921 rpy=-3.141492 3.141923 2.847039, axis 0 0 1
- added joint caster_freeJoint__167__: type continuous, parent caster_link__166__, child caster_wheel__168__, origin xyz=0.010622 0.003223 -0.015539 rpy=-1.570796 3.141593 -2.847039, axis 0 0 1
- added joint leftMotor__162__: type continuous, parent base_link, child leftWheel__163__, origin xyz=0.022255 0.082750 -0.020626 rpy=1.570796 3.141938 -3.141593, axis 0 0 1
- added joint rightMotor__159__: type continuous, parent base_link, child rightWheel__160__, origin xyz=0.022257 -0.082751 -0.020637 rpy=1.570796 3.141938 -3.141592, axis 0 0 1
