Commit message: Remove inertia component from urdf file

File: ros2_ws/scripts/resources/models/mazebot.urdf (robot description, URDF)
Before this commit: robot PioneerP3DX__158__, 5 links, 4 joints
Links:
- link base_link: mass 2.0 -> None
- link caster_link__166__: mass 0.125 -> None
- link caster_wheel__168__: mass 0.03125 -> None
- link leftWheel__163__: mass 0.1875 -> None
- link rightWheel__160__: mass 0.1875 -> None
