Commit message: Change joint names for mazebot urdf model

File: ros2_ws/src/mazebot/models/mazebot.urdf (robot description, URDF)
Before this commit: robot PioneerP3DX__158__, 5 links, 4 joints
Joints:
- removed joint caster_freeJoint__165__
- removed joint caster_freeJoint__167__
- removed joint leftMotor__162__
- removed joint rightMotor__159__
- added joint caster_freeJoint1: type continuous, parent base_link, child caster_link__166__, origin xyz=-0.074513 -0.000001 -0.038921 rpy=-3.141492 3.141923 2.847039, axis 0 0 1
- added joint caster_freeJoint2: type continuous, parent caster_link__166__, child caster_wheel__168__, origin xyz=0.010622 0.003223 -0.015539 rpy=-1.570796 3.141593 -2.847039, axis 0 0 1
- added joint leftMotor: type continuous, parent base_link, child leftWheel__163__, origin xyz=0.022255 0.082750 -0.020626 rpy=1.570796 3.141938 -3.141593, axis 0 0 1
- added joint rightMotor: type continuous, parent base_link, child rightWheel__160__, origin xyz=0.022257 -0.082751 -0.020637 rpy=1.570796 3.141938 -3.141592, axis 0 0 1
